Commit message: working multicam

File: multicam/simple_kinect_model2_twoCameras.xacro (robot description, xacro)
@@ -47,8 +47,4 @@
       <axis xyz="0 1 0" />
       <origin xyz="0.027 0.0 1.10" rpy="0.0 0.2 0"/>
-  </joint>
-    <joint name="world_jnt" type="fixed">
-      <parent link="world"/>
-      <child link="base_link"/>
   </joint>
     <link name="kinect_link2">
